File: trapapoul/proto_uno/Arduino_As_Uno.sch (KiCad schematic (older format))
At the start: 75 parts, among them J1 MICROSD, K1 CONN_3, P1 Power, P10 CONN_2, P11 CONN_2, P12 CONN_3X2, P2 Analog, P3 Digital, P4 Digital, P5 CONN_01X01, P6 CONN_01X01, P7 CONN_01X01, P8 CONN_01X01, P9 CONN_4, Q1 PBSS5350, Q2 PMV16XN, Q3 DSS20200L, Q4 DMP1045U, Q5 DMP1045U, Q6 PBSS4320, U1 TL431LP, U2 MCP7940, U3 CAT24C64, U4 MIC5205, U5 MIC5205, U6 aop, X1 32.768KHz

Commit message: before rooting
pcb a été préparé
Parts:
- removed Q1: PBSS5350, ~, symbol PNP
- removed Q2: PMV16XN, ~, symbol NPN
- removed Q3: DSS20200L, ~, symbol PNP
- removed Q4, Q5: DMP1045U, ~, symbol PNP
- removed Q6: PBSS4320, ~, symbol NPN
- added C18: 100n, Capacitors_ThroughHole:C_Disc_D7.5_P5, symbol C-RESCUE-Arduino_As_Uno
- added Q1, Q3, Q4, Q5: PBSS5350, TO_SOT_Packages_SMD:SOT-23_Handsoldering, symbol PNP_3-Term
- added Q2, Q6: PBSS4320, TO_SOT_Packages_SMD:SOT-23_Handsoldering, symbol NPN_3-Term
- C1, C2: value C -> 10p; footprint ~ -> Capacitors_ThroughHole:C_Disc_D6_P5
- C10, C8, C9: value 100uF -> 100u; footprint ~ -> Capacitors_ThroughHole:C_Radial_D10_L13_P5
- C11, C12, C13, C16, C17, C3, C7: footprint ~ -> Capacitors_ThroughHole:C_Disc_D12_P7.75
- C14: value 470pF -> 470p; footprint ~ -> Capacitors_ThroughHole:C_Disc_D6_P5
- C15: footprint ~ -> Capacitors_ThroughHole:C_Disc_D6_P5
- C4: value 100nF -> 100n; footprint ~ -> Capacitors_ThroughHole:C_Disc_D12_P7.75
- C5: value 100nF -> 100n; footprint ~ -> Capacitors_ThroughHole:C_Disc_D7.5_P5
- C6: value 1u -> 100n; footprint ~ -> Capacitors_ThroughHole:C_Disc_D7.5_P5
- F1, F2: footprint ~ -> Resistors_ThroughHole:Resistor_Horizontal_RM15mm
- J1: footprint ~ -> Connect:SD_Card_Receptacle
- K1: footprint (none) -> Connect:bornier3
- P10, P11: footprint (none) -> Connect:bornier2
- P12: footprint (none) -> Connectors_Molex:Molex_Microfit3_Header_02x03_Straight_43045-0628
- P9: footprint (none) -> Connect:bornier4
- R1, R10, R11, R12, R13, R14, R15, R16, R17, R18, R19, R2, R20, R21, R22, R23, R24, R25, R26, R3, R4, R5, R6, R7, R8, R9: footprint ~ -> Resistors_ThroughHole:Resistor_Horizontal_RM10mm
- RV1, RV2: footprint ~ -> Potentiometers:Potentiometer_Triwood_RM-065
- SP1: footprint ~ -> Connect:bornier2
- U1: footprint SOT23 -> TO_SOT_Packages_SMD:SOT-23
- U2, U6: footprint (none) -> Housings_DIP:DIP-8_W7.62mm_LongPads
- U3: footprint ~ -> Housings_DIP:DIP-8_W7.62mm_LongPads
- U4, U5: footprint (none) -> TO_SOT_Packages_SMD:SOT-23-5
- X1: footprint ~ -> Crystals:Crystal_HC49-U_Horizontal_Typ1
Connections:
- wire segments 181 -> 135
Other:
- moved on the sheet: C1, C2, C3, C4, C5, C6, F1, F2, J1, K1, P10, P9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
