File: trapapoul/proto_uno/Arduino_As_Uno.kicad_pcb (KiCad board)
At the start: 2 copper layers, 68.6 x 53.3 mm, 76 parts, among them J1 MICROSD, K1 CONN_3, P1 Power, P10 CONN_2, P11 CONN_2, P12 CONN_3X2, P2 Analog, P3 Digital, P4 Digital, P5 CONN_01X01, P6 CONN_01X01, P7 CONN_01X01, P8 CONN_01X01, P9 CONN_4, Q1 PBSS5350, Q2 PBSS4320, Q3 PBSS5350, Q4 PBSS5350, Q5 PBSS5350, Q6 PBSS4320, U1 TL431LP, U2 MCP7940, U3 CAT24C64, U4 MIC5205, U5 MIC5205, U6 aop, X1 32.768KHz

Commit message: unknown changes
Parts:
- removed C10, C8, C9: 100u, Capacitors_ThroughHole:C_Radial_D10_L13_P5
- removed C11, C12, C13, C16, C17, C7: 1u, Capacitors_ThroughHole:C_Disc_D12_P7.75
- removed C14: 470p, Capacitors_ThroughHole:C_Disc_D6_P5
- removed C15: 470pF, Capacitors_ThroughHole:C_Disc_D6_P5
- removed C18, C5, C6: 100n, Capacitors_ThroughHole:C_Disc_D7.5_P5
- removed C3: 100nF, Capacitors_ThroughHole:C_Disc_D12_P7.75
- removed C4: 100n, Capacitors_ThroughHole:C_Disc_D12_P7.75
- removed F1: 1A, Resistors_ThroughHole:Resistor_Horizontal_RM15mm
- removed F2: 3A, Resistors_ThroughHole:Resistor_Horizontal_RM15mm
- removed K1: CONN_3, Connect:bornier3
- removed P10, P11: CONN_2, Connect:bornier2
- removed P12: CONN_3X2, Connectors_Molex:Molex_Microfit3_Header_02x03_Straight_43045-0628
- removed P9: CONN_4, Connect:bornier4
- removed Q1, Q3, Q4, Q5: PBSS5350, TO_SOT_Packages_SMD:SOT-23
- removed Q2, Q6: PBSS4320, TO_SOT_Packages_SMD:SOT-23
- removed R1: 100k, Resistors_ThroughHole:Resistor_Horizontal_RM10mm
- removed R10, R11, R12, R13, R14, R16, R17, R2, R22, R3, R7, R9: 10k, Resistors_ThroughHole:Resistor_Horizontal_RM10mm
- removed R15, R18, R21, R25: 100, Resistors_ThroughHole:Resistor_Horizontal_RM10mm
- removed R19, R20, R23, R24, R8: 1k, Resistors_ThroughHole:Resistor_Horizontal_RM10mm
- removed R26: 0.2, Resistors_ThroughHole:Resistor_Horizontal_RM10mm
- removed R4: 4k7, Resistors_ThroughHole:Resistor_Horizontal_RM10mm
- removed R5, R6: 2.2k, Resistors_ThroughHole:Resistor_Horizontal_RM10mm
- removed RV1, RV2: 200k, Potentiometers:Potentiometer_Triwood_RM-065
- removed SP1: SPEAKER, Connect:bornier2
- removed U2: MCP7940, Housings_DIP:DIP-8_W7.62mm_LongPads
- removed U3: CAT24C64, Housings_DIP:DIP-8_W7.62mm_LongPads
- removed U4, U5: MIC5205, TO_SOT_Packages_SMD:SOT-23-5
- removed U6: aop, Housings_DIP:DIP-8_W7.62mm_LongPads
- removed X1: 32.768KHz, Crystals:Crystal_HC49-U_Horizontal_Typ1
- added C201: 1u, Capacitors_ThroughHole:C_Radial_D5_L11_P2, F.Cu at (169.0, 42.9)
- added C203: 1u, Capacitors_ThroughHole:C_Radial_D5_L11_P2, F.Cu at (164.0, 39.9)
- added C205: 1u, Capacitors_ThroughHole:C_Radial_D5_L11_P2, F.Cu at (169.0, 36.9)
- added C301: 1u, Capacitors_ThroughHole:C_Radial_D5_L11_P2, F.Cu at (79.0, 97.4)
- added C302: 1u, Capacitors_ThroughHole:C_Radial_D5_L11_P2, F.Cu at (87.0, 97.4)
- added C303: 470pF, Capacitors_ThroughHole:C_Disc_D6_P5, F.Cu at (92.0, 92.4)
- added C311: 1u, Capacitors_ThroughHole:C_Radial_D5_L11_P2, F.Cu at (51.5, 95.4)
- added C312: 1u, Capacitors_ThroughHole:C_Radial_D5_L11_P2, F.Cu at (59.0, 95.4)
- added C313: 470p, Capacitors_ThroughHole:C_Disc_D6_P5, F.Cu at (64.0, 90.9)
- added C401: 100u, Capacitors_ThroughHole:C_Radial_D10_L13_P5, F.Cu at (144.0, 152.9)
- added C402: 100u, Capacitors_ThroughHole:C_Radial_D10_L13_P5, F.Cu at (155.0, 144.9)
- added C403: 100u, Capacitors_ThroughHole:C_Radial_D10_L13_P5, F.Cu at (144.5, 141.9)
- added C500: 100n, Capacitors_ThroughHole:C_Disc_D7.5_P5, F.Cu at (54.0, 123.4)
- added C501: 10p, Capacitors_ThroughHole:C_Disc_D6_P5, F.Cu at (40.0, 118.4)
- added C502: 10p, Capacitors_ThroughHole:C_Disc_D6_P5, F.Cu at (48.0, 118.4)
- added C600: 100nF, Capacitors_ThroughHole:C_Disc_D12_P7.75, F.Cu at (140.0, 115.9)
- added C700: 100n, Capacitors_ThroughHole:C_Disc_D12_P7.75, F.Cu at (124.0, 111.4)
- added F600: 1A, Resistors_ThroughHole:Resistor_Horizontal_RM15mm, F.Cu at (135.5, 113.9)
- added F700: 3A, Resistors_ThroughHole:Resistor_Horizontal_RM15mm, F.Cu at (132.0, 113.9)
- added J201: CONN_3X2, Pin_Headers:Pin_Header_Straight_2x03, F.Cu at (171.0, 53.9)
- added J3: CONN_4, Pin_Headers:Pin_Header_Straight_1x04, F.Cu at (131.5, 87.9)
- added J4: CONN_2, Pin_Headers:Pin_Header_Straight_1x02, F.Cu at (128.0, 79.9)
- added J6: CONN_2, Terminal_Blocks:TerminalBlock_Pheonix_MKDS1.5-2pol, F.Cu at (134.5, 120.4)
- added J7: CONN_3, Terminal_Blocks:TerminalBlock_Pheonix_MKDS1.5-3pol, F.Cu at (116.5, 123.4)
- added Q101: PBSS5350, TO_SOT_Packages_SMD:SOT-23_Handsoldering, F.Cu at (219.5, 99.9)
- added Q102: PBSS5350, TO_SOT_Packages_SMD:SOT-23_Handsoldering, F.Cu at (216.5, 103.9)
- added Q103: PBSS4320, TO_SOT_Packages_SMD:SOT-23_Handsoldering, F.Cu at (216.5, 96.9)
- added Q104: PBSS5350, TO_SOT_Packages_SMD:SOT-23_Handsoldering, F.Cu at (205.0, 101.9)
- added Q105: PBSS5350, TO_SOT_Packages_SMD:SOT-23_Handsoldering, F.Cu at (208.5, 104.9)
- added Q106: PBSS4320, TO_SOT_Packages_SMD:SOT-23_Handsoldering, F.Cu at (201.5, 103.9)
- added R101: 100, Resistors_ThroughHole:Resistor_Horizontal_RM10mm, F.Cu at (210.0, 98.4)
- added R102: 1k, Resistors_ThroughHole:Resistor_Horizontal_RM10mm, F.Cu at (213.0, 105.4)
- added R103: 100, Resistors_ThroughHole:Resistor_Horizontal_RM10mm, F.Cu at (213.0, 89.4)
- added R104: 100, Resistors_ThroughHole:Resistor_Horizontal_RM10mm, F.Cu at (200.0, 95.4)
- added R105: 1k, Resistors_ThroughHole:Resistor_Horizontal_RM10mm, F.Cu at (210.0, 108.4)
- added R106: 100, Resistors_ThroughHole:Resistor_Horizontal_RM10mm, F.Cu at (210.0, 89.4)
- added R107: 10k, Resistors_ThroughHole:Resistor_Horizontal_RM10mm, F.Cu at (223.0, 92.4)
- added R108: 10k, Resistors_ThroughHole:Resistor_Horizontal_RM10mm, F.Cu at (200.0, 92.4)
- added R110: 10k, Resistors_ThroughHole:Resistor_Horizontal_RM10mm, F.Cu at (235.7, 97.1)
- added R111: 1k, Resistors_ThroughHole:Resistor_Horizontal_RM10mm, F.Cu at (229.7, 97.1)
- added R112: 1k, Resistors_ThroughHole:Resistor_Horizontal_RM10mm, F.Cu at (232.7, 97.1)
- added R113: 0.2, Resistors_ThroughHole:Resistor_Horizontal_RM10mm, F.Cu at (226.2, 107.1)
- added R201: 10k, Resistors_ThroughHole:Resistor_Horizontal_RM10mm, F.Cu at (180.2, 44.9)
- added R202: 10k, Resistors_ThroughHole:Resistor_Horizontal_RM10mm, F.Cu at (180.2, 56.7)
- added R203: 10k, Resistors_ThroughHole:Resistor_Horizontal_RM10mm, F.Cu at (177.6, 44.9)
- added R204: 10k, Resistors_ThroughHole:Resistor_Horizontal_RM10mm, F.Cu at (177.6, 56.7)
- added R205: 10k, Resistors_ThroughHole:Resistor_Horizontal_RM10mm, F.Cu at (175.0, 44.9)
- added R206: 10k, Resistors_ThroughHole:Resistor_Horizontal_RM10mm, F.Cu at (175.0, 56.7)
- added R301: 1k, Resistors_ThroughHole:Resistor_Horizontal_RM10mm, F.Cu at (89.0, 87.4)
- added R311: 10k, Resistors_ThroughHole:Resistor_Horizontal_RM10mm, F.Cu at (61.0, 85.9)
- added R450: 100k, Resistors_ThroughHole:Resistor_Horizontal_RM10mm, F.Cu at (135.0, 88.4)
- added R501: 10k, Resistors_ThroughHole:Resistor_Horizontal_RM10mm, F.Cu at (55.0, 126.4)
- added R502: 2.2k, Resistors_ThroughHole:Resistor_Horizontal_RM10mm, F.Cu at (52.0, 126.4)
- added R503: 2.2k, Resistors_ThroughHole:Resistor_Horizontal_RM10mm, F.Cu at (49.0, 126.4)
- added R701: 10k, Resistors_ThroughHole:Resistor_Horizontal_RM10mm, F.Cu at (125.0, 97.4)
- added R702: 4k7, Resistors_ThroughHole:Resistor_Horizontal_RM10mm, F.Cu at (128.5, 103.9)
- added RV301: 200k, Potentiometers:Potentiometer_Triwood_RM-065, F.Cu at (90.0, 99.4)
- added RV311: 200k, Potentiometers:Potentiometer_Triwood_RM-065, F.Cu at (62.0, 98.4)
- added SP4: SPEAKER, Connect:bornier2, F.Cu at (157.5, 154.4)
- added U110: aop, Housings_DIP:DIP-8_W7.62mm_LongPads, F.Cu at (234.7, 110.1)
- added U301: MIC5205, TO_SOT_Packages_SMD:SOT-23-5, F.Cu at (83.0, 94.9)
- added U302: MIC1825, TO_SOT_Packages_THT:Pentawatt_Neutral_Straight_Vertical_TO220-5-T05A, F.Cu at (83.0, 92.4)
- added U311: MIC5205, TO_SOT_Packages_SMD:SOT-23-5, F.Cu at (55.0, 92.9)
- added U312: MIC1825, TO_SOT_Packages_THT:Pentawatt_Neutral_Straight_Vertical_TO220-5-T05A, F.Cu at (55.0, 90.4)
- added U400: CAT24C64, Housings_DIP:DIP-8_W7.62mm_LongPads, F.Cu at (121.5, 74.9)
- added U450: TL431LP, TO_SOT_Packages_SMD:SOT-23, F.Cu at (133.5, 78.4)
- added U500: MCP7940, Housings_DIP:DIP-8_W7.62mm_LongPads, F.Cu at (38.3, 127.4)
- added X500: 32.768KHz, Crystals:Crystal_Round_Horizontal_3mm_BigPad, F.Cu at (44.0, 123.4)
- C1, C2: value 10p -> 100n; footprint Capacitors_ThroughHole:C_Disc_D6_P5 -> Capacitors_ThroughHole:C_Disc_D7.5_P5
- U1: value TL431LP -> TL431TH; footprint TO_SOT_Packages_SMD:SOT-23 -> TO_SOT_Packages_THT:TO-92_Inline_Narrow_Oval
- moved J1 141.6 mm to (136.0, 20.4)
- moved C2 104.0 mm to (152.0, 120.9), turned to 180 degrees
- moved U1 101.3 mm to (138.0, 78.4), turned to 270 degrees
- moved C1 55.8 mm to (139.0, 120.9)
Connections:
- C1 pad 2: Net-(C1-Pad2) -> +3.3V
- C2 pad 2: Net-(C2-Pad2) -> +5V
- J1 pad 1: Net-(J1-Pad1) -> (no net)
- J1 pad 8: Net-(J1-Pad8) -> (no net)
- P1 pad 1: Net-(P1-Pad1) -> (no net)
- P1 pad 2: /IOREF -> (no net)
- P1 pad 3: /Reset -> (no net)
- P1 pad 8: /Vin -> (no net)
- P2 pad 1: Mes_lux -> (no net)
- P2 pad 4: /A3 -> (no net)
- P3 pad 10: /8 -> (no net)
- P4 pad 1: /7 -> (no net)
- P5 pad 1: Net-(P5-Pad1) -> (no net)
- P6 pad 1: Net-(P6-Pad1) -> (no net)
- P7 pad 1: Net-(P7-Pad1) -> (no net)
- P8 pad 1: Net-(P8-Pad1) -> (no net)
- U1 pad 1: Net-(U1-Pad1) -> A_REF
- U1 pad 2: A_REF -> GND
- U1 pad 3: GND -> A_REF
Routing:
- net GND: track 0.00 -> 25.2 mm
- net Net-(J201-Pad1): track 0.00 -> 14.7 mm
- net BUTTON_UP: track 0.00 -> 13.8 mm
- net BUTTON_MID: track 0.00 -> 13.7 mm
- net Net-(J201-Pad3): track 0.00 -> 11.4 mm
- net Net-(J201-Pad5): track 0.00 -> 6.66 mm
- net +3.3V: track 0.00 -> 5.20 mm
- net BUTTON_LOW: track 0.00 -> 4.89 mm
Other:
- net class Default: clearance 0.2 -> 0.3; trace_width 0.25 -> 0.5; via_dia 0.6 -> 1.5; via_drill 0.4 -> 0.8
- rule trace_clearance: 0.2 -> 0.3
