File: trapapoul/proto_ptibou/Arduino_As_Uno.sch (KiCad schematic (older format))
At the start: 80 parts, among them J1 MICROSD, J201 CONN_3X2, J3 CONN_4, J4 CONN_2, J6 CONN_2, J7 CONN_3, P1 Power, P2 Analog, P3 Digital, P4 Digital, P5 CONN_01X01, P6 CONN_01X01, P7 CONN_01X01, P8 CONN_01X01, Q101 PBSS5350, Q102 PBSS5350, Q103 PBSS4320, Q104 PBSS5350, Q105 PBSS5350, Q106 PBSS4320, U1 TL431TH, U110 aop, U301 MIC5205, U302 MIC1825, U311 MIC5205, U312 MIC1825, U400 CAT24C64, U450 TL431LP, U500 MCP7940, X500 32.768KHz

Commit message: unknown changes
Parts:
- removed C401, C402, C403: 100u, Capacitors_ThroughHole:C_Radial_D10_L13_P5, symbol C-RESCUE-Arduino_As_Uno
- removed J1: MICROSD, Connect:SD_Card_Receptacle, symbol MicroSD
- removed J4: CONN_2, Pin_Headers:Pin_Header_Straight_1x02, symbol CONN_2
- removed Q101, Q102, Q104, Q105: PBSS5350, TO_SOT_Packages_SMD:SOT-23_Handsoldering, symbol PNP_3-Term
- removed Q103, Q106: PBSS4320, TO_SOT_Packages_SMD:SOT-23_Handsoldering, symbol NPN_3-Term
- removed R101, R103, R104, R106: 100, Resistors_ThroughHole:Resistor_Horizontal_RM10mm, symbol R-RESCUE-Arduino_As_Uno
- removed R102, R105, R111, R112: 1k, Resistors_ThroughHole:Resistor_Horizontal_RM10mm, symbol R-RESCUE-Arduino_As_Uno
- removed R107, R108, R110: 10k, Resistors_ThroughHole:Resistor_Horizontal_RM10mm, symbol R-RESCUE-Arduino_As_Uno
- removed R113: 0.2, Resistors_ThroughHole:Resistor_Horizontal_RM10mm, symbol R-RESCUE-Arduino_As_Uno
- removed SP4: SPEAKER, Connect:bornier2, symbol SPEAKER
- removed U110: aop, Housings_DIP:DIP-8_W7.62mm_LongPads, symbol LM2903small
- removed U400: CAT24C64, Housings_DIP:DIP-8_W7.62mm_LongPads, symbol CAT24C64
- added J4: CONN_01X06, Pin_Headers:Pin_Header_Straight_1x06, symbol CONN_01X06
Connections:
- net labels removed: MOT_A, MOT_B
- wire segments 139 -> 93
- no-connect marks 8 -> 2
Other:
- note removed: "Buzzer"
- note removed: "Memoire EEprom"
- note removed: "Pont en H"
- note removed: "adr=1010000"
