File: trapapoul/proto_traparduino/proto_traparduino.sch (KiCad schematic (older format))
At the start: 89 parts, among them P1 Power, P2 Analog, P3 Digital, P4 Digital, P5 CONN_1, P6 CONN_1, P7 CONN_1, P8 CONN_1

Commit message: trapapoul_proto2 fini
Parts:
- removed C? (x10): C, symbol C
- removed D?: SCHOTTKY, symbol SCHOTTKY
- removed P1: Power, Socket_Arduino_Uno:Socket_Strip_Arduino_1x08, symbol CONN_8
- removed P2: Analog, Socket_Arduino_Uno:Socket_Strip_Arduino_1x06, symbol CONN_6
- removed P3: Digital, Socket_Arduino_Uno:Socket_Strip_Arduino_1x10, symbol CONN_10
- removed P4: Digital, Socket_Arduino_Uno:Socket_Strip_Arduino_1x08, symbol CONN_8
- removed P5, P6, P7, P8: CONN_1, Socket_Arduino_Uno:Arduino_1pin, symbol CONN_1
- removed R?: POT, symbol POT
- removed R?: R, symbol R
- removed U?: MIC5205, symbol MIC5205
- added C203: 10n, Capacitors_SMD:C_1206_HandSoldering, symbol C
- added C302, C303, C304, C305, C306, C307, C308, C309: 10uF, Capacitors_SMD:C_1206_HandSoldering, symbol C
- added C310, C710: 220u, Capacitors_ThroughHole:C_Radial_D7.5_L11.2_P2.5, symbol cap
- added C702, C712: 1n, Capacitors_SMD:C_1206_HandSoldering, symbol C
- added C703, C713, C830: 100n, Capacitors_SMD:C_1206_HandSoldering, symbol C
- added C711, C714: 10u, Capacitors_SMD:C_1206_HandSoldering, symbol C
- added D711: SCHOTTKY, Diodes_SMD:MiniMELF_Handsoldering, symbol SCHOTTKY
- added J800: HEADER_2, Pin_Headers:Pin_Header_Straight_1x02, symbol HEADER_2
- added R711: 10k, Resistors_SMD:R_1206_HandSoldering, symbol R
- added RP71: 100k, Potentiometers:Potentiometer_Triwood_RM-065, symbol POT
- added U711: MIC5205, TO_SOT_Packages_SMD:SOT-23-5, symbol MIC5205
- C201, C202: renamed from C?; value C -> 10p; footprint (none) -> Capacitors_SMD:C_1206_HandSoldering
- C301: renamed from C?; value C -> 10uF; footprint (none) -> Capacitors_SMD:C_1206_HandSoldering
- C401, C402, C403, C721, C725: renamed from C?; value C -> 10n; footprint (none) -> Capacitors_SMD:C_1206_HandSoldering
- C602, C612: renamed from C?; value C -> 100nF; footprint (none) -> Capacitors_SMD:C_1206_HandSoldering
- C701, C704: renamed from C?; value C -> 10u; footprint (none) -> Capacitors_SMD:C_1206_HandSoldering
- C705, C715: renamed from C?; value cap -> 220u; footprint (none) -> Capacitors_ThroughHole:C_Radial_D7.5_L11.2_P2.5
- C831: renamed from C?; value C -> 100n; footprint (none) -> Capacitors_SMD:C_1206_HandSoldering
- D701: renamed from D?; footprint (none) -> Diodes_SMD:MELF_Handsoldering
- F721: renamed from F?; value FUSE -> 5A; footprint (none) -> Fuse_Holders_and_Fuses:Fuse_SMD1206_HandSoldering
- J000: renamed from J?; footprint (none) -> w_conn_misc:arduino_header
- J400, J740: renamed from J?; footprint (none) -> Pin_Headers:Pin_Header_Straight_1x04
- J720, J730: renamed from J?; footprint (none) -> Pin_Headers:Pin_Header_Straight_1x02
- Q811, Q821: renamed from Q?; value NPN_BEC -> PBSS4320; footprint (none) -> TO_SOT_Packages_SMD:SOT-23_Handsoldering
- Q812, Q813, Q822, Q823: renamed from Q?; value PNP_BEC -> PBSS5350; footprint (none) -> TO_SOT_Packages_SMD:SOT-23_Handsoldering
- R201, R401, R402, R403, R701, R721, R722, R724, R731, R732: renamed from R?; value R -> 10k; footprint (none) -> Resistors_SMD:R_1206_HandSoldering
- R202, R203: renamed from R?; value R -> 2.2k; footprint (none) -> Resistors_SMD:R_1206_HandSoldering
- R601, R602, R611, R612, R811, R812, R813, R821, R822, R823, R831, R832, R833, R834: renamed from R?; footprint (none) -> Resistors_SMD:R_1206_HandSoldering
- R810, R820: renamed from R?; value 330 -> 3k3; footprint (none) -> Resistors_SMD:R_1206_HandSoldering
- R835: renamed from R?; value 0.2 -> 0R2; footprint (none) -> Resistors_SMD:R_1206_HandSoldering
- RP70: renamed from R?; value POT -> 100k; footprint (none) -> Potentiometers:Potentiometer_Triwood_RM-065
- RP72: renamed from R?; value POT -> 10k; footprint (none) -> Potentiometers:Potentiometer_Triwood_RM-065
- U201: renamed from U?; footprint (none) -> SMD_Packages:SOIC-8-N
- U300: renamed from BZ?; footprint (none) -> Buzzers_Beepers:Buzzer_12x9.5RM7.6
- U601, U611: renamed from U?; footprint (none) -> gdi:ITR9606
- U701, U830: renamed from U?; footprint (none) -> TO_SOT_Packages_SMD:SOT-23-5
- U725: renamed from D?; footprint (none) -> TO_SOT_Packages_SMD:SOT-23_Handsoldering
- X201: renamed from X?; value CRYSTAL -> 32.768K; footprint (none) -> Crystals:Crystal_Round_Vertical_3mm_BigPad
Connections:
- net labels removed: +3.3V, +3V3, +5V, 0(Rx), 1(Tx), 10(**/SS), 11(**/MOSI), 12(MISO), 13(SCK), 2, 3(**), 4, 5(**), 6(**), 7, 8, 9(**), A0, A1, A2, A3, A4(SDA), A5(SCL), AREF, IOREF, Reset, Vin
- wire segments 145 -> 149
- no-connect marks 5 -> 0
Other:
- note added: "5.4V"
- note added: "cmp lib\nis reversed"
- note removed: "Holes"
- note removed: "Shield for Arduino that uses\nthe same pin disposition\nlike "Uno" board Rev 3."
- moved on the sheet: C201, C202, C301, C401, C402, C403, C602, C612, C701, C704, C705, C715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
