File: trapapoul/proto_trapapoul_4/_autosave-proto_trapapoul4.kicad_pcb (KiCad board)
At the start: 2 copper layers, 113 x 48 mm, 118 parts, among them J101 HEADER_4x2, J401 HEADER_2, J402 HEADER_2, J403 HEADER_2, J730 HEADER_2, J801 HEADER_1, J802 HEADER_1, J901 HEADER_6, J902 HEADER_6, Q811 NPN, Q812 PNP, Q821 NPN, Q822 PNP, Q900 NPN, U100 ATMEGA328P-A, U201 MCP7940, U500 MIC5205, U510 MIC5205, U520 MIC5205, U603 A3144, U604 A3144, U715 431, U830 MCP601-SOT, U900 PCF8574, X104 16M, X201 32.768K

Commit message: reconnect
Parts:
- R501: moved to B.Cu
- turned R501 to 90 degrees
Changed lines of the file:
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@@
   (general
     (links 252)
-    (no_connects 2)
+    (no_connects 4)
     (area 101.234762 50.043039 215.950001 101.9)
     (thickness 1.6)
@@
     (34 B.Paste user hide)
     (35 F.Paste user hide)
-    (36 B.SilkS user)
+    (36 B.SilkS user hide)
     (37 F.SilkS user hide)
     (38 B.Mask user hide)
@@
     (46 B.CrtYd user hide)
     (47 F.CrtYd user hide)
-    (48 B.Fab user)
+    (48 B.Fab user hide)
     (49 F.Fab user hide)
   )
@@
     )
   )
-  (module Resistors_SMD:R_1206 (layer F.Cu)
-    (at 183.2 64.7 270)
+  (module Resistors_SMD:R_1206 (layer B.Cu)
+    (at 183.2 64.7 90)
     (descr "Resistor SMD 1206, reflow soldering, Vishay (see dcrcw.pdf)")
     (tags "resistor 1206")
     (attr smd)
-    (fp_text reference R501 (at 0 -2.3 270) (layer F.SilkS)
-      (effects (font (size 1 1) (thickness 0.15)))
+    (fp_text reference R501 (at 0 2.3 90) (layer B.SilkS)
+      (effects (font (size 1 1) (thickness 0.15)) (justify mirror))
     )
-    (fp_text value 47k (at 0.1 -0.1 270) (layer F.Fab)
-      (effects (font (size 1 1) (thickness 0.15)))
+    (fp_text value 47k (at 0.1 0.1 90) (layer B.Fab)
+      (effects (font (size 1 1) (thickness 0.15)) (justify mirror))
     )
-    (fp_line (start -1.6 0.8) (end -1.6 -0.8) (layer F.Fab) (width 0.1))
-    (fp_line (start 1.6 0.8) (end -1.6 0.8) (layer F.Fab) (width 0.1))
-    (fp_line (start 1.6 -0.8) (end 1.6 0.8) (layer F.Fab) (width 0.1))
-    (fp_line (start -1.6 -0.8) (end 1.6 -0.8) (layer F.Fab) (width 0.1))
-    (fp_line (start -2.2 -1.2) (end 2.2 -1.2) (layer F.CrtYd) (width 0.05))
-    (fp_line (start -2.2 1.2) (end 2.2 1.2) (layer F.CrtYd) (width 0.05))
-    (fp_line (start -2.2 -1.2) (end -2.2 1.2) (layer F.CrtYd) (width 0.05))
-    (fp_line (start 2.2 -1.2) (end 2.2 1.2) (layer F.CrtYd) (width 0.05))
-    (fp_line (start 1 1.075) (end -1 1.075) (layer F.SilkS) (width 0.15))
-    (fp_line (start -1 -1.075) (end 1 -1.075) (layer F.SilkS) (width 0.15))
-    (pad 1 smd rect (at -1.45 0 270) (size 0.9 1.7) (layers F.Cu F.Paste F.Mask)
+    (fp_line (start -1.6 -0.8) (end -1.6 0.8) (layer B.Fab) (width 0.1))
+    (fp_line (start 1.6 -0.8) (end -1.6 -0.8) (layer B.Fab) (width 0.1))
+    (fp_line (start 1.6 0.8) (end 1.6 -0.8) (layer B.Fab) (width 0.1))
+    (fp_line (start -1.6 0.8) (end 1.6 0.8) (layer B.Fab) (width 0.1))
+    (fp_line (start -2.2 1.2) (end 2.2 1.2) (layer B.CrtYd) (width 0.05))
+    (fp_line (start -2.2 -1.2) (end 2.2 -1.2) (layer B.CrtYd) (width 0.05))
+    (fp_line (start -2.2 1.2) (end -2.2 -1.2) (layer B.CrtYd) (width 0.05))
+    (fp_line (start 2.2 1.2) (end 2.2 -1.2) (layer B.CrtYd) (width 0.05))
+    (fp_line (start 1 -1.075) (end -1 -1.075) (layer B.SilkS) (width 0.15))
+    (fp_line (start -1 1.075) (end 1 1.075) (layer B.SilkS) (width 0.15))
+    (pad 1 smd rect (at -1.45 0 90) (size 0.9 1.7) (layers B.Cu B.Paste B.Mask)
       (net 14 "Net-(C503-Pad1)"))
-    (pad 2 smd rect (at 1.45 0 270) (size 0.9 1.7) (layers F.Cu F.Paste F.Mask)
+    (pad 2 smd rect (at 1.45 0 90) (size 0.9 1.7) (layers B.Cu B.Paste B.Mask)
       (net 2 GND))
     (model Resistors_SMD.3dshapes/R_1206.wrl
