File: trapapoul/proto_trapapoul_4/proto_trapapoul4.sch (KiCad schematic (older format))
At the start: 116 parts, among them J101 HEADER_3x2, J401 HEADER_2, J402 HEADER_2, J403 HEADER_2, J410 HEADER_4, J730 HEADER_2, J801 HEADER_1, J802 HEADER_1, J901 HEADER_6, J902 HEADER_6, Q811 PBSS4320, Q812 PBSS5350, Q821 PBSS4320, Q822 PBSS5350, Q900 PBSS4320, U100 ATMEGA328P-A, U201 MCP7940, U500 MIC5205, U510 MIC5205, U520 MIC5205, U601 A3144, U602 A3144, U603 A3144, U604 A3144, U715 TLV431-DBZ, U830 MCP601-SOT, U900 PCF8574, X104 16M, X201 32.768K

Commit message: prototrapapoul4 un peu retouché
Parts:
- removed C103, C541, C710: 10n, Capacitors_SMD:C_1206, symbol C
- removed C543: 10uF, Capacitors_SMD:C_1206, symbol C
- removed J101: HEADER_3x2, Pin_Headers:Pin_Header_Straight_2x03, symbol HEADER_3x2
- removed J410: HEADER_4, Pin_Headers:Pin_Header_Angled_1x04, symbol HEADER_4
- removed R505, R506: tbd, Resistors_SMD:R_1206, symbol R
- removed U601, U602: A3144, TO_SOT_Packages_THT:TO-92_Inline_Narrow_Oval, symbol A3144
- added C106, C107, C108, C109: 100nF, Capacitors_SMD:C_1206, symbol C
- added H901, H902, H903, H904: hole, gdi:3mm_screw, symbol hole
- added J101: HEADER_4x2, Pin_Headers:Pin_Header_Straight_2x04_Pitch2.54mm, symbol HEADER_4x2
- added R501, R513, R713: 47k, Resistors_SMD:R_1206, symbol R
- added R502: 10k, Resistors_SMD:R_1206, symbol R
- C101, C203, C401, C402, C403: value 10n -> 100nF
- C102, C830, C831: value 100n -> 100nF
- C104, C105, C201, C202: value 10p -> 10pF
- C503, C513, C522: value 470p -> 470pF
- C732: renamed from C502; value 10n -> 100nF
- C901: value 10nF -> 100nF
- R203, R204: value 2.2k -> 2k2
- R500, R832: value 10k -> 47k
- R512: value 33k -> 47k
- R525: value tbd -> 10k
- R526: value tbd -> 47k
- R602, R612: value 4k7 -> 10k
- R712: value 4.7k -> 47k
- R721: value 4.7k -> 100k
- R722, R731: value 10k -> 100k
- R732: value 2.2k -> 47k
- R810, R820: value 3k3 -> 2k2
- R831: value 1k -> 10k
- R902: value 4.7k -> 10k
- X104: footprint Crystals:Crystal_HC49-U_Vertical -> Crystals:Crystal_HC49-SD_SMD
Connections:
- wire segments 310 -> 334
Other:
- note added: "13V*147/47=4.15"
- note added: "2.5V/57*104=4.55v"
- note added: "400mA*0.2Ohm*48=3.84V"
- note added: "i*dt=C*dU => t=470uF*1V/15mA=31ms"
- note added: "tau=10K*100NF=1ms"
- note removed: "41"
- moved on the sheet: C732, R711, R712, U715

Commit message: reconnect
Parts:
- C101, C102, C104, C105, C106, C107, C108, C109, C201, C202, C203, C401, C402, C403, C501, C503, C504, C512, C513, C514, C521, C522, C523, C531, C542, C602, C612, C722, C732, C830, C831, C900, C901, C902: symbol C -> C-RESCUE-proto_trapapoul4
- F721: symbol FUSE -> FUSE-RESCUE-proto_trapapoul4
- Q811, Q821, Q900: value PBSS4320 -> NPN
- Q812, Q822: value PBSS5350 -> PNP
- R201, R203, R204, R401, R402, R403, R500, R501, R502, R510, R511, R512, R513, R520, R525, R526, R602, R612, R711, R712, R713, R714, R721, R722, R731, R732, R810, R811, R812, R820, R821, R822, R831, R832, R833, R834, R835, R902: symbol R -> R-RESCUE-proto_trapapoul4
- RP90: symbol POT -> POT-RESCUE-proto_trapapoul4
- U900: symbol PCF8574 -> PCF8574-RESCUE-proto_trapapoul4
